File: IrrigationValve/kicad/IrrigationValveMOSFET/IrrigationValve.sch (KiCad schematic (older format))
At the start: 10 parts, among them CON1 BARREL_JACK, Q1 IRL540N, U1 arduino_nano

Commit message: kicad
Parts:
- RV1: symbol POT -> POT-RESCUE-IrrigationValve
Changed lines of the file:
@@
 NoConn ~ 3650 5500
 $Comp
-L POT RV1
+L POT-RESCUE-IrrigationValve RV1
 U 1 1 55E93CB9
 P 1600 4000
